Commit message: Foxy to Humble upgrades

File: description/robot_core.xacro (robot description, xacro)
@@ -637,7 +637,7 @@
         <origin rpy="0 0 0" xyz="0.2259 0 0.0438" />
         <parent link="chassis"/>
-        <child link="sonar_front"/>
-    </joint>
-    <link name="sonar_front">
+        <child link="base_sonar_front"/>
+    </joint>
+    <link name="base_sonar_front">
         <collision>
         <origin xyz="0.001975 0 0.0038" rpy="0 0 0"/>
@@ -658,5 +658,5 @@
         </inertial>
     </link>
-    <gazebo reference="sonar_front">
+    <gazebo reference="base_sonar_front">
         <sensor type="ray" name="TeraRanger">
             <pose>0 0 0 0 0 0</pose>

Commit message: Navigation issues

File: description/robot_core.xacro (robot description, xacro)
@@ -253,383 +253,4 @@
         <mu2 value="0.001"/>
     </gazebo>
-    <!-- TOP SONAR -->
-    <!--SONAR 1-->
-    <joint name="sonar_front_1_joint" type="fixed">
-        <axis xyz="0 1 0" />
-        <origin rpy="0 0 0" xyz="0.15 0 0.671" />
-        <parent link="chassis"/>
-        <child link="sonar_top_1"/>
-    </joint>
-    <link name="sonar_top_1">
-        <collision>
-        <origin xyz="0 0 0" rpy="0 0 0"/>
-        <geometry>
-            <box size="0.01 0.01 0.01"/>
-        </geometry>
-        </collision>
-        <visual>
-        <origin xyz="0 0 0" rpy="0 0 0"/>
-        <geometry>
-            <box size="0.01 0.01 0.01"/>
-        </geometry>
-        </visual>
-        <inertial>
-        <mass value="1e-5" />
-        <origin xyz="0 0 0" rpy="0 0 0"/>
-        <inertia ixx="1e-6" ixy="0" ixz="0" iyy="1e-6" iyz="0" izz="1e-6" />
-        </inertial>
-    </link>
-    <gazebo reference="sonar_top_1">
-    <sensor type="ray" name="TeraRanger">
-        <pose>0 0 0 0 0 0</pose>
-        <visualize>true</visualize>
-        <update_rate>50</update_rate>
-        <ray>
-            <scan>
-                <horizontal>
-                <samples>10</samples>
-                <resolution>1</resolution>
-                <min_angle>-0.14835</min_angle>
-                <max_angle>0.14835</max_angle>
-                </horizontal>
-                <vertical>
-                <samples>10</samples>
-                <resolution>1</resolution>
-                <min_angle>-0.14835</min_angle>
-                <max_angle>0.14835</max_angle>
-                </vertical>
-            </scan>
-            <range>
-                <min>0.01</min>
-                <max>2</max>
-                <resolution>0.02</resolution>
-            </range>
-        </ray>
-        <plugin filename="libgazebo_ros_range.so" name="gazebo_ros_range">
-            <gaussianNoise>0.005</gaussianNoise>
-            <alwaysOn>true</alwaysOn>
-            <updateRate>50</updateRate>
-            <topicName>sensor/Range</topicName>
-            <frameName>sonar_top_1</frameName>
-            <radiation>INFRARED</radiation>
-            <fov>0.2967</fov>
-        </plugin>
-    </sensor>
-    </gazebo>
-     <!--SONAR 2-->
-    <joint name="sonar_front_2_joint" type="fixed">
-        <axis xyz="0 1 0" />
-        <origin rpy="0 0 0" xyz="0.15 0 0.5948" />
-        <parent link="chassis"/>
-        <child link="sonar_top_2"/>
-    </joint>
-    <link name="sonar_top_2">
-        <collision>
-        <origin xyz="0 0 0" rpy="0 0 0"/>
-        <geometry>
-            <box size="0.01 0.01 0.01"/>
-        </geometry>
-        </collision>
-        <visual>
-        <origin xyz="0 0 0" rpy="0 0 0"/>
-        <geometry>
-            <box size="0.01 0.01 0.01"/>
-        </geometry>
-        </visual>
-        <inertial>
-        <mass value="1e-5" />
-        <origin xyz="0 0 0" rpy="0 0 0"/>
-        <inertia ixx="1e-6" ixy="0" ixz="0" iyy="1e-6" iyz="0" izz="1e-6" />
-        </inertial>
-    </link>
-    <gazebo reference="sonar_top_2">
-        <sensor type="ray" name="TeraRanger">
-            <pose>0 0 0 0 0 0</pose>
-            <visualize>true</visualize>
-            <update_rate>50</update_rate>
-            <ray>
-                <scan>
-                    <horizontal>
-                    <samples>10</samples>
-                    <resolution>1</resolution>
-                    <min_angle>-0.14835</min_angle>
-                    <max_angle>0.14835</max_angle>
-                    </horizontal>
-                    <vertical>
-                    <samples>10</samples>
-                    <resolution>1</resolution>
-                    <min_angle>-0.14835</min_angle>
-                    <max_angle>0.14835</max_angle>
-                    </vertical>
-                </scan>
-                <range>
-                    <min>0.01</min>
-                    <max>2</max>
-                    <resolution>0.02</resolution>
-                </range>
-            </ray>
-            <plugin filename="libgazebo_ros_range.so" name="ultrasonic_sensor_2">
-                <gaussianNoise>0.005</gaussianNoise>
-                <alwaysOn>true</alwaysOn>
-                <updateRate>50</updateRate>
-                <topicName>sensor_msgs/range_2</topicName>
-                <frameName>sonar_top_2</frameName>
-                <radiation>ultrasound</radiation>
-                <fov>0.2967</fov>
-            </plugin>
-        </sensor>
-    </gazebo>
-     <!--SONAR 3-->
-    <joint name="sonar_front_3_joint" type="fixed">
-        <axis xyz="0 1 0" />
-        <origin rpy="0 0 0" xyz="0.15 0 0.5186" />
-        <parent link="chassis"/>
-        <child link="sonar_top_3"/>
-    </joint>
-    <link name="sonar_top_3">
-        <collision>
-        <origin xyz="0 0 0" rpy="0 0 0"/>
-        <geometry>
-            <box size="0.01 0.01 0.01"/>
-        </geometry>
-        </collision>
-        <visual>
-        <origin xyz="0 0 0" rpy="0 0 0"/>
-        <geometry>
-            <box size="0.01 0.01 0.01"/>
-        </geometry>
-        </visual>
-        <inertial>
-        <mass value="1e-5" />
-        <origin xyz="0 0 0" rpy="0 0 0"/>
-        <inertia ixx="1e-6" ixy="0" ixz="0" iyy="1e-6" iyz="0" izz="1e-6" />
-        </inertial>
-    </link>
-    <gazebo reference="sonar_top_3">
-        <sensor type="ray" name="TeraRanger">
-            <pose>0 0 0 0 0 0</pose>
-            <visualize>true</visualize>
-            <update_rate>50</update_rate>
-            <ray>
-                <scan>
-                    <horizontal>
-                    <samples>10</samples>
-                    <resolution>1</resolution>
-                    <min_angle>-0.14835</min_angle>
-                    <max_angle>0.14835</max_angle>
-                    </horizontal>
-                    <vertical>
-                    <samples>10</samples>
-                    <resolution>1</resolution>
-                    <min_angle>-0.14835</min_angle>
-                    <max_angle>0.14835</max_angle>
-                    </vertical>
-                </scan>
-                <range>
-                    <min>0.01</min>
-                    <max>2</max>
-                    <resolution>0.02</resolution>
-                </range>
-            </ray>
-            <plugin filename="libgazebo_ros_range.so" name="ultrasonic_sensor_3">
-                <gaussianNoise>0.005</gaussianNoise>
-                <alwaysOn>true</alwaysOn>
-                <updateRate>50</updateRate>
-                <topicName>sensor_msgs/range_3</topicName>
-                <frameName>sonar_top</frameName>
-                <radiation>ultrasound</radiation>
-                <fov>0.2967</fov>
-            </plugin>
-        </sensor>
-    </gazebo>
-     <!--SONAR 4-->
-    <joint name="sonar_front_4_joint" type="fixed">
-        <axis xyz="0 1 0" />
-        <origin rpy="0 0 0" xyz="0.15 0 0.4424" />
-        <parent link="chassis"/>
-        <child link="sonar_top_4"/>
-    </joint>
-    <link name="sonar_top_4">
-        <collision>
-        <origin xyz="0 0 0" rpy="0 0 0"/>
-        <geometry>
-            <box size="0.01 0.01 0.01"/>
-        </geometry>
-        </collision>
-        <visual>
-        <origin xyz="0 0 0" rpy="0 0 0"/>
-        <geometry>
-            <box size="0.01 0.01 0.01"/>
-        </geometry>
-        </visual>
-        <inertial>
-        <mass value="1e-5" />
-        <origin xyz="0 0 0" rpy="0 0 0"/>
-        <inertia ixx="1e-6" ixy="0" ixz="0" iyy="1e-6" iyz="0" izz="1e-6" />
-        </inertial>
-    </link>
-    <gazebo reference="sonar_top_4">
-        <sensor type="ray" name="TeraRanger">
-            <pose>0 0 0 0 0 0</pose>
-            <visualize>true</visualize>
-            <update_rate>50</update_rate>
-            <ray>
-                <scan>
-                    <horizontal>
-                    <samples>10</samples>
-                    <resolution>1</resolution>
-                    <min_angle>-0.14835</min_angle>
-                    <max_angle>0.14835</max_angle>
-                    </horizontal>
-                    <vertical>
-                    <samples>10</samples>
-                    <resolution>1</resolution>
-                    <min_angle>-0.14835</min_angle>
-                    <max_angle>0.14835</max_angle>
-                    </vertical>
-                </scan>
-                <range>
-                    <min>0.01</min>
-                    <max>2</max>
-                    <resolution>0.02</resolution>
-                </range>
-            </ray>
-            <plugin filename="libgazebo_ros_range.so" name="ultrasonic_sensor_4">
-                <gaussianNoise>0.005</gaussianNoise>
-                <alwaysOn>true</alwaysOn>
-                <updateRate>50</updateRate>
-                <topicName>sensor_msgs/range_4</topicName>
-                <frameName>sonar_top</frameName>
-                <radiation>ultrasound</radiation>
-                <fov>0.2967</fov>
-            </plugin>
-        </sensor>
-    </gazebo>
-     <!--SONAR 5-->
-    <joint name="sonar_front_5_joint" type="fixed">
-        <axis xyz="0 1 0" />
-        <origin rpy="0 0 0" xyz="0.15 0 0.3662" />
-        <parent link="chassis"/>
-        <child link="sonar_top_5"/>
-    </joint>
-    <link name="sonar_top_5">
-        <collision>
-        <origin xyz="0 0 0" rpy="0 0 0"/>
-        <geometry>
-            <box size="0.01 0.01 0.01"/>
-        </geometry>
-        </collision>
-        <visual>
-        <origin xyz="0 0 0" rpy="0 0 0"/>
-        <geometry>
-            <box size="0.01 0.01 0.01"/>
-        </geometry>
-        </visual>
-        <inertial>
-        <mass value="1e-5" />
-        <origin xyz="0 0 0" rpy="0 0 0"/>
-        <inertia ixx="1e-6" ixy="0" ixz="0" iyy="1e-6" iyz="0" izz="1e-6" />
-        </inertial>
-    </link>
-    <gazebo reference="sonar_top_5">
-        <sensor type="ray" name="TeraRanger">
-            <pose>0 0 0 0 0 0</pose>
-            <visualize>true</visualize>
-            <update_rate>50</update_rate>
-            <ray>
-                <scan>
-                    <horizontal>
-                    <samples>10</samples>
-                    <resolution>1</resolution>
-                    <min_angle>-0.14835</min_angle>
-                    <max_angle>0.14835</max_angle>
-                    </horizontal>
-                    <vertical>
-                    <samples>10</samples>
-                    <resolution>1</resolution>
-                    <min_angle>-0.14835</min_angle>
-                    <max_angle>0.14835</max_angle>
-                    </vertical>
-                </scan>
-                <range>
-                    <min>0.01</min>
-                    <max>2</max>
-                    <resolution>0.02</resolution>
-                </range>
-            </ray>
-            <plugin filename="libgazebo_ros_range.so" name="ultrasonic_sensor_5">
-                <gaussianNoise>0.005</gaussianNoise>
-                <alwaysOn>true</alwaysOn>
-                <updateRate>50</updateRate>
-                <topicName>sensor_msgs/range_5</topicName>
-                <frameName>sonar_top</frameName>
-                <radiation>ultrasound</radiation>
-                <fov>0.2967</fov>
-            </plugin>
-        </sensor>
-    </gazebo>
-     <!--SONAR 6-->
-    <joint name="sonar_front_6_joint" type="fixed">
-        <axis xyz="0 1 0" />
-        <origin rpy="0 0 0" xyz="0.15 0 0.29" />
-        <parent link="chassis"/>
-        <child link="sonar_top_6"/>
-    </joint>
-    <link name="sonar_top_6">
-        <collision>
-        <origin xyz="0.15 0 0.29" rpy="0 0 0"/>
-        <geometry>
-            <box size="0.01 0.01 0.01"/>
-        </geometry>
-        </collision>
-        <visual>
-        <origin xyz="0 0 0" rpy="0 0 0"/>
-        <geometry>
-            <box size="0.01 0.01 0.01"/>
-        </geometry>
-        </visual>
-        <inertial>
-        <mass value="1e-5" />
-        <origin xyz="0 0 0" rpy="0 0 0"/>
-        <inertia ixx="1e-6" ixy="0" ixz="0" iyy="1e-6" iyz="0" izz="1e-6" />
-        </inertial>
-    </link>
-    <gazebo reference="sonar_top_6">
-        <sensor type="ray" name="TeraRanger">
-            <pose>0 0 0 0 0 0</pose>
-            <visualize>true</visualize>
-            <update_rate>50</update_rate>
-            <ray>
-                <scan>
-                    <horizontal>
-                    <samples>10</samples>
-                    <resolution>1</resolution>
-                    <min_angle>-0.14835</min_angle>
-                    <max_angle>0.14835</max_angle>
-                    </horizontal>
-                    <vertical>
-                    <samples>10</samples>
-                    <resolution>1</resolution>
-                    <min_angle>-0.14835</min_angle>
-                    <max_angle>0.14835</max_angle>
-                    </vertical>
-                </scan>
-                <range>
-                    <min>0.01</min>
-                    <max>2</max>
-                    <resolution>0.02</resolution>
-                </range>
-            </ray>
-            <plugin filename="libgazebo_ros_range.so" name="ultrasonic_sensor_6">
-                <gaussianNoise>0.005</gaussianNoise>
-                <alwaysOn>true</alwaysOn>
-                <updateRate>50</updateRate>
-                <topicName>sensor_msgs/range_6</topicName>
-                <frameName>sonar_top</frameName>
-                <radiation>ultrasound</radiation>
-                <fov>0.2967</fov>
-            </plugin>
-        </sensor>
-    </gazebo>
      <!--SONAR TOP LEFT FRONT-->
     <joint name="sonar_left_top_joint" type="fixed">

Commit message: Added gazebo ref to casters

File: description/robot_core.xacro (robot description, xacro)
@@ -176,4 +176,9 @@
         </xacro:inertial_cylinder>
     </link>
+    <gazebo reference="front_caster_swivel">
+        <material>Gazebo/Blue</material>
+        <mu1 value="0.001"/>
+        <mu2 value="0.001"/>
+    </gazebo>
     <joint name="front_caster_wheel_joint" type="continuous">
         <parent link="front_caster_swivel"/>
@@ -226,4 +231,9 @@
         </xacro:inertial_cylinder>
     </link>
+    <gazebo reference="rear_caster_swivel">
+        <material>Gazebo/Blue</material>
+        <mu1 value="0.001"/>
+        <mu2 value="0.001"/>
+    </gazebo>
     <joint name="rear_caster_wheel_joint" type="continuous">
         <parent link="rear_caster_swivel"/>
@@ -248,5 +258,5 @@
         </xacro:inertial_cylinder>
     </link>
-    <gazebo reference="caster_wheel">
+    <gazebo reference="rear_caster_wheel">
         <material>Gazebo/Blue</material>
         <mu1 value="0.001"/>
@@ -305,5 +315,5 @@
                 </range>
             </ray>
-            <plugin filename="libgazebo_ros_range.so" name="ultrasonic_sensor_7">
+            <plugin filename="libgazebo_ros_range.so" name="base_sonar_left_top">
                 <gaussianNoise>0.005</gaussianNoise>
                 <alwaysOn>true</alwaysOn>
@@ -368,5 +378,5 @@
                 </range>
             </ray>
-            <plugin filename="libgazebo_ros_range.so" name="ultrasonic_sensor_8">
+            <plugin filename="libgazebo_ros_range.so" name="base_sonar_left_bottom">
                 <gaussianNoise>0.005</gaussianNoise>
                 <alwaysOn>true</alwaysOn>
@@ -431,5 +441,5 @@
                 </range>
             </ray>
-            <plugin filename="libgazebo_ros_range.so" name="ultrasonic_sensor_9">
+            <plugin filename="libgazebo_ros_range.so" name="base_sonar_right_top">
                 <gaussianNoise>0.005</gaussianNoise>
                 <alwaysOn>true</alwaysOn>
@@ -494,5 +504,5 @@
                 </range>
             </ray>
-            <plugin filename="libgazebo_ros_range.so" name="ultrasonic_sensor_10">
+            <plugin filename="libgazebo_ros_range.so" name="base_sonar_right_bottom">
                 <gaussianNoise>0.005</gaussianNoise>
                 <alwaysOn>true</alwaysOn>
