Commit message: Change lidar configuration

File: description/lidar.xacro (robot description, xacro)
@@ -1,8 +1,29 @@
 <?xml version="1.0"?>
 <robot xmlns:xacro="http://www.ros.org/wiki/xacro" >
+    <joint name="laser_mount_joint" type="fixed">
+        <parent link="chassis"/>
+        <child link="laser_mount_frame"/>
+        <origin xyz="0 0 0.78" rpy="0 0 0"/>
+    </joint>
+    <link name="laser_mount_frame">
+        <visual>
+            <geometry>
+                <cylinder radius="0.02" length="0.24"/>
+            </geometry>
+            <material name="black"/>
+        </visual>
+        <collision>
+            <geometry>
+                <cylinder radius="0.05" length="0.04"/>
+            </geometry>
+        </collision>
+        <xacro:inertial_cylinder mass="0.1" length="0.04" radius="0.05">
+            <origin xyz="0 0 0" rpy="0 0 0"/>
+        </xacro:inertial_cylinder>
+    </link>
     <joint name="laser_joint" type="fixed">
         <parent link="chassis"/>
         <child link="laser_frame"/>
-        <origin xyz="0 0 0.76" rpy="0 0 0"/>
+        <origin xyz="0 0 0.91" rpy="0.7 0 0"/>
     </joint>
     <link name="laser_frame">

File: description/robot_core.xacro (robot description, xacro)
@@ -98,5 +98,5 @@
         </xacro:inertial_cylinder>
     </link>
-    <gazebo reference="chassis">
+    <gazebo reference="body">
         <material>Gazebo/White</material>
     </gazebo>
@@ -632,12 +632,12 @@
         </sensor>
     </gazebo>
-     <!--SONAR BASE FRONT-->
-    <joint name="sonar_front_joint" type="fixed">
-        <axis xyz="0 1 0" />
-        <origin rpy="0 0 0" xyz="0.2259 0 0.0438" />
-        <parent link="chassis"/>
-        <child link="base_sonar_front"/>
-    </joint>
-    <link name="base_sonar_front">
+     <!--SONAR TOP LEFT FRONT-->
+    <joint name="sonar_left_top_joint" type="fixed">
+        <axis xyz="0 1 0" />
+        <origin rpy="0 0 0.60" xyz="0.193 0.12 0.09" />
+        <parent link="chassis"/>
+        <child link="base_sonar_left_top"/>
+    </joint>
+    <link name="base_sonar_left_top">
         <collision>
         <origin xyz="0.001975 0 0.0038" rpy="0 0 0"/>
@@ -658,5 +658,5 @@
         </inertial>
     </link>
-    <gazebo reference="base_sonar_front">
+    <gazebo reference="base_sonar_left_top">
         <sensor type="ray" name="TeraRanger">
             <pose>0 0 0 0 0 0</pose>
@@ -688,5 +688,5 @@
                 <alwaysOn>true</alwaysOn>
                 <updateRate>50</updateRate>
-                <topicName>sensor_msgs/range_front</topicName>
+                <topicName>sensor_msgs/range_left_top</topicName>
                 <frameName>sonar_base</frameName>
                 <radiation>ultrasound</radiation>
@@ -696,30 +696,30 @@
     </gazebo>
 <!-- LEFT SONAR -->
-    <joint name="sonar_left_joint" type="fixed">
-        <axis xyz="0 1 0" />
-        <origin rpy="0 0 1.57" xyz="0 0.2259 0.0438" />
-        <parent link="chassis"/>
-        <child link="base_sonar_left"/>
-    </joint>
-    <link name="base_sonar_left">
-        <collision>
-        <origin xyz="0 0 0" rpy="0 0 0"/>
-        <geometry>
-            <box size="0.01 0.01 0.01"/>
-        </geometry>
-        </collision>
-        <visual>
-        <origin xyz="0 0 0" rpy="0 0 0"/>
-        <geometry>
-            <box size="0.01 0.01 0.01"/>
-        </geometry>
-        </visual>
-        <inertial>
-        <mass value="1e-5" />
-        <origin xyz="0 0 0" rpy="0 0 0"/>
-        <inertia ixx="1e-6" ixy="0" ixz="0" iyy="1e-6" iyz="0" izz="1e-6" />
-        </inertial>
-    </link>
-    <gazebo reference="base_sonar_left">
+    <joint name="sonar_left_bottom_joint" type="fixed">
+        <axis xyz="0 1 0" />
+        <origin rpy="0 0 0.60" xyz="0.18 0.14 0.00001" />
+        <parent link="chassis"/>
+        <child link="base_sonar_left_bottom"/>
+    </joint>
+    <link name="base_sonar_left_bottom">
+        <collision>
+        <origin xyz="0 0 0" rpy="0 0 0"/>
+        <geometry>
+            <box size="0.01 0.01 0.01"/>
+        </geometry>
+        </collision>
+        <visual>
+        <origin xyz="0 0 0" rpy="0 0 0"/>
+        <geometry>
+            <box size="0.01 0.01 0.01"/>
+        </geometry>
+        </visual>
+        <inertial>
+        <mass value="1e-5" />
+        <origin xyz="0 0 0" rpy="0 0 0"/>
+        <inertia ixx="1e-6" ixy="0" ixz="0" iyy="1e-6" iyz="0" izz="1e-6" />
+        </inertial>
+    </link>
+    <gazebo reference="base_sonar_left_bottom">
         <sensor type="ray" name="TeraRanger">
             <pose>0 0 0 0 0 0</pose>
@@ -751,5 +751,5 @@
                 <alwaysOn>true</alwaysOn>
                 <updateRate>50</updateRate>
-                <topicName>sensor_msgs/range_left</topicName>
+                <topicName>sensor_msgs/range_left_bottom</topicName>
                 <frameName>sonar_base</frameName>
                 <radiation>ultrasound</radiation>
@@ -759,30 +759,30 @@
     </gazebo>
 <!-- RIGHT SONAR  -->
-    <joint name="sonar_right_joint" type="fixed">
-        <axis xyz="0 1 0" />
-        <origin rpy="0 0 -1.57" xyz="0 -0.2259 0.0438" />
-        <parent link="chassis"/>
-        <child link="base_sonar_right"/>
-    </joint>
-    <link name="base_sonar_right">
-        <collision>
-        <origin xyz="0 0 0" rpy="0 0 0"/>
-        <geometry>
-            <box size="0.01 0.01 0.01"/>
-        </geometry>
-        </collision>
-        <visual>
-        <origin xyz="0 0 0" rpy="0 0 0"/>
-        <geometry>
-            <box size="0.01 0.01 0.01"/>
-        </geometry>
-        </visual>
-        <inertial>
-        <mass value="1e-5" />
-        <origin xyz="0 0 0" rpy="0 0 0"/>
-        <inertia ixx="1e-6" ixy="0" ixz="0" iyy="1e-6" iyz="0" izz="1e-6" />
-        </inertial>
-    </link>
-    <gazebo reference="base_sonar_right">
+    <joint name="sonar_right_top_joint" type="fixed">
+        <axis xyz="0 1 0" />
+        <origin rpy="0 0 -0.60" xyz="0.193 -0.12 0.09" />
+        <parent link="chassis"/>
+        <child link="base_sonar_right_top"/>
+    </joint>
+    <link name="base_sonar_right_top">
+        <collision>
+        <origin xyz="0 0 0" rpy="0 0 0"/>
+        <geometry>
+            <box size="0.01 0.01 0.01"/>
+        </geometry>
+        </collision>
+        <visual>
+        <origin xyz="0 0 0" rpy="0 0 0"/>
+        <geometry>
+            <box size="0.01 0.01 0.01"/>
+        </geometry>
+        </visual>
+        <inertial>
+        <mass value="1e-5" />
+        <origin xyz="0 0 0" rpy="0 0 0"/>
+        <inertia ixx="1e-6" ixy="0" ixz="0" iyy="1e-6" iyz="0" izz="1e-6" />
+        </inertial>
+    </link>
+    <gazebo reference="base_sonar_right_top">
         <sensor type="ray" name="TeraRanger">
             <pose>0 0 0 0 0 0</pose>
@@ -814,5 +814,5 @@
                 <alwaysOn>true</alwaysOn>
                 <updateRate>50</updateRate>
-                <topicName>sensor_msgs/range_right</topicName>
+                <topicName>sensor_msgs/range_right_top</topicName>
                 <frameName>sonar_base</frameName>
                 <radiation>ultrasound</radiation>
@@ -822,30 +822,30 @@
     </gazebo>
 <!-- REAR SONAR  -->
-    <joint name="sonar_rear_joint" type="fixed">
-        <axis xyz="0 1 0" />
-        <origin rpy="0 0 -3.14" xyz="-0.227 0 0.0438" />
-        <parent link="chassis"/>
-        <child link="base_sonar_rear"/>
-    </joint>
-    <link name="base_sonar_rear">
-        <collision>
-        <origin xyz="0 0 0" rpy="0 0 0"/>
-        <geometry>
-            <box size="0.01 0.01 0.01"/>
-        </geometry>
-        </collision>
-        <visual>
-        <origin xyz="0 0 0" rpy="0 0 0"/>
-        <geometry>
-            <box size="0.01 0.01 0.01"/>
-        </geometry>
-        </visual>
-        <inertial>
-        <mass value="1e-5" />
-        <origin xyz="0 0 0" rpy="0 0 0"/>
-        <inertia ixx="1e-6" ixy="0" ixz="0" iyy="1e-6" iyz="0" izz="1e-6" />
-        </inertial>
-    </link>
-    <gazebo reference="base_sonar_rear">
+    <joint name="sonar_right_bottom_joint" type="fixed">
+        <axis xyz="0 1 0" />
+        <origin rpy="0 0 -0.60" xyz="0.18 -0.14 0.00001" />
+        <parent link="chassis"/>
+        <child link="base_sonar_right_bottom"/>
+    </joint>
+    <link name="base_sonar_right_bottom">
+        <collision>
+        <origin xyz="0 0 0" rpy="0 0 0"/>
+        <geometry>
+            <box size="0.01 0.01 0.01"/>
+        </geometry>
+        </collision>
+        <visual>
+        <origin xyz="0 0 0" rpy="0 0 0"/>
+        <geometry>
+            <box size="0.01 0.01 0.01"/>
+        </geometry>
+        </visual>
+        <inertial>
+        <mass value="1e-5" />
+        <origin xyz="0 0 0" rpy="0 0 0"/>
+        <inertia ixx="1e-6" ixy="0" ixz="0" iyy="1e-6" iyz="0" izz="1e-6" />
+        </inertial>
+    </link>
+    <gazebo reference="base_sonar_right_bottom">
         <sensor type="ray" name="TeraRanger">
             <pose>0 0 0 0 0 0</pose>
@@ -877,10 +877,7 @@
                 <alwaysOn>true</alwaysOn>
                 <updateRate>50</updateRate>
-                <ros>
-                    <remapping>~/out:=ultrasonic_sensor_10</remapping>
-                </ros>
-                <output_type>sensor_msgs/Range</output_type>
+                <output_type>sensor_msgs/range_right_bottom</output_type>
                 <radiation_type>ultrasound</radiation_type>
-                <frame_name>base_sonar_rear</frame_name>
+                <frame_name>sonar_base</frame_name>
                 <fov>0.2967</fov>
             </plugin>

Commit message: Set laser back to level

File: description/lidar.xacro (robot description, xacro)
@@ -1,29 +1,8 @@
 <?xml version="1.0"?>
 <robot xmlns:xacro="http://www.ros.org/wiki/xacro" >
-    <joint name="laser_mount_joint" type="fixed">
-        <parent link="chassis"/>
-        <child link="laser_mount_frame"/>
-        <origin xyz="0 0 0.78" rpy="0 0 0"/>
-    </joint>
-    <link name="laser_mount_frame">
-        <visual>
-            <geometry>
-                <cylinder radius="0.02" length="0.24"/>
-            </geometry>
-            <material name="black"/>
-        </visual>
-        <collision>
-            <geometry>
-                <cylinder radius="0.05" length="0.04"/>
-            </geometry>
-        </collision>
-        <xacro:inertial_cylinder mass="0.1" length="0.04" radius="0.05">
-            <origin xyz="0 0 0" rpy="0 0 0"/>
-        </xacro:inertial_cylinder>
-    </link>
     <joint name="laser_joint" type="fixed">
         <parent link="chassis"/>
         <child link="laser_frame"/>
-        <origin xyz="0 0 0.91" rpy="0.7 0 0"/>
+        <origin xyz="0 0 0.91" rpy="0 0 0"/>
     </joint>
     <link name="laser_frame">

Commit message: Added base_footprint

File: description/lidar.xacro (robot description, xacro)
@@ -4,5 +4,5 @@
         <parent link="chassis"/>
         <child link="laser_frame"/>
-        <origin xyz="0 0 0.91" rpy="0 0 0"/>
+        <origin xyz="0 0 0.76" rpy="0 0 0"/>
     </joint>
     <link name="laser_frame">

File: description/robot_core.xacro (robot description, xacro)
@@ -20,4 +20,12 @@
     <link name="base_link">
     </link>
+    <!-- BASE_FOOTPRINT LINK -->
+    <joint name="base_footprint_joint" type="fixed">
+        <parent link="base_link"/>
+        <child link="base_footprint"/>
+        <origin xyz="0 0 0" rpy="0 0 0"/>
+    </joint>
+    <link name="base_footprint">
+    </link>
     <!-- CHASSIS LINK -->
     <joint name="chassis_joint" type="fixed">
